File: ysws by viperkeebs/ysws by viperkeebs.kicad_pcb (KiCad board)
At the start: 2 copper layers, 69.8 x 94 mm, 19 parts, among them U1 Arduino_Pro_Micro

Commit message: :3
Parts:
- moved U1 17.3 mm to (119.1, 47.3)
Routing:
- net Col 1: track 78.0 -> 57.5 mm, vias 0 -> 1
- net Col 3: track 58.2 -> 69.5 mm
- net Row 1: track 63.6 -> 68.5 mm
- net Row 2: track 84.6 -> 81.5 mm, vias 0 -> 1
- net Row 3: track 102.2 -> 104.5 mm
- net Col 2: track 60.4 -> 59.7 mm
- added copper zone on B.Cu, net (none)
- added copper zone on F.Cu, net (none)
Other:
- outline, holes or cut-outs redrawn
